Commit message: Update yahboomcar_R2.urdf

File: src/rosmaster_description/urdf/yahboomcar_R2.urdf (robot description, URDF)
Before this commit: robot yahboomcar, 9 links, 8 joints
Links:
- link back_left_link: geometry collision mesh filename=package://rosmaster_description/meshes/back_right_link.STL; visual mesh filename=package://rosmaster_description/meshes/back_right_link.STL
- link back_right_link: geometry collision mesh filename=package://rosmaster_description/meshes/back_right_link.STL; visual mesh filename=package://rosmaster_description/meshes/back_right_link.STL
- link base_link: geometry collision mesh filename=package://rosmaster_description/meshes/base_link.STL; visual mesh filename=package://rosmaster_description/meshes/base_link.STL
- link camera_link: geometry collision mesh filename=package://rosmaster_description/meshes/camera_link_R2.STL; visual mesh filename=package://rosmaster_description/meshes/camera_link_R2.STL
- link front_left_steer: geometry collision mesh filename=package://rosmaster_description/meshes/front_left_steer.STL; visual mesh filename=package://rosmaster_description/meshes/front_left_steer.STL
- link front_left_wheel: geometry collision mesh filename=package://rosmaster_description/meshes/back_right_link.STL; visual mesh filename=package://rosmaster_description/meshes/back_right_link.STL
- link front_right_steer: geometry collision mesh filename=package://rosmaster_description/meshes/front_left_steer.STL; visual mesh filename=package://rosmaster_description/meshes/front_left_steer.STL
- link front_right_wheel: geometry collision mesh filename=package://rosmaster_description/meshes/back_right_link.STL; visual mesh filename=package://rosmaster_description/meshes/back_right_link.STL
- link laser_link: geometry collision mesh filename=package://rosmaster_description/meshes/laser_link_R2.STL; visual mesh filename=package://rosmaster_description/meshes/laser_link_R2.STL
